File: hardware/pcb/usbc.kicad_sch (KiCad schematic)
At the start: 6 parts, among them J48 USB_C_Receptacle_USB2.0_16P, U53 CH334R, U54 USBLC6-2SC6

Commit message: fix : le décalage de références corrompait la feuille usbc
Mon script de copie décalait toute chaîne de la forme lettre+chiffre, pas
seulement les références. Sur usbc (offset +40), il a donc transformé :

  (paper "A4")  ->  "A44"   -> KiCad : « Page type non valide, ligne 6 »
  les noms de pins de l'USB-C : A1->A41, CC1->CC41, SBU1->SBU41, VDD33->VDD73

D'où la feuille qui s'ouvrait vide et l'échec de chargement des feuilles
hiérarchiques.

Le décalage ne s'applique plus qu'aux vraies références, et seulement là où
elles sont déclarées : (property "Reference" "U13") et (reference "U13") dans
les blocs d'instances. Copie refaite : paper A4 rétabli, noms de pins intacts,
seules C13/J8/R50/R52/U13/U14 décalées en C53/J48/R90/R92/U53/U54.

Les feuilles power et mcu n'étaient pas touchées (offset 0, aucune substitution).
ERC : 0 erreur, 96 warnings (liens de bibliothèque).

Co-Authored-By: Claude Opus 5 <noreply@anthropic.com>
Claude-Session: https://claude.ai/code/session_01GfX5RmekmQi78Dm37qsT4Z
Connections:
- net +5V: now also J48.A4 (VBUS), J48.A9 (VBUS), J48.B4 (VBUS), J48.B9 (VBUS); no longer J48.A44 (VBUS), J48.A49 (VBUS), J48.B44 (VBUS), J48.B49 (VBUS)
- net GND: now also J48.A1 (GND), J48.A12 (GND), J48.B1 (GND), J48.B12 (GND); no longer J48.A41 (GND), J48.A52 (GND), J48.B41 (GND), J48.B52 (GND)
- net at R92.2: now also J48.B5 (CC2); no longer J48.B45 (CC42)
- net at R90.1: now also J48.A5 (CC1); no longer J48.A45 (CC41)
- new net: J48.A7 (D-), J48.B7 (D-), U54.1 (I/O1)
- new net: J48.A6 (D+), J48.B6 (D+), U54.3 (I/O2)
Changed lines of the file:
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@@
 	(generator "eeschema")
 	(generator_version "10.0")
-	(paper "A44")
+	(paper "A4")
 	(junction
 		(at 69.85 166.37)
@@
 			)
 		)
-		(pin "B47"
-		)
-		(pin "A52"
+		(pin "B7"
+		)
+		(pin "A12"
 		)
 		(pin "SH"
 		)
-		(pin "B48"
-		)
-		(pin "A49"
-		)
-		(pin "B46"
-		)
-		(pin "A41"
-		)
-		(pin "B44"
-		)
-		(pin "B49"
-		)
-		(pin "A48"
-		)
-		(pin "B45"
-		)
-		(pin "B52"
-		)
-		(pin "B41"
-		)
-		(pin "A46"
-		)
-		(pin "A47"
-		)
-		(pin "A45"
-		)
-		(pin "A44"
+		(pin "B8"
+		)
+		(pin "A9"
+		)
+		(pin "B6"
+		)
+		(pin "A1"
+		)
+		(pin "B4"
+		)
+		(pin "B9"
+		)
+		(pin "A8"
+		)
+		(pin "B5"
+		)
+		(pin "B12"
+		)
+		(pin "B1"
+		)
+		(pin "A6"
+		)
+		(pin "A7"
+		)
+		(pin "A5"
+		)
+		(pin "A4"
 		)
 		(instances
