File: hardware/pcb/usbc.kicad_sch (KiCad schematic)
At the start: 6 parts, among them J48 USB_C_Receptacle_USB2.0_16P, U53 CH334R, U54 USBLC6-2SC6

Commit message: élagage des feuilles + réparation des tables de bibliothèques
Mae a élagué dans l'éditeur :
- mcu  : 108 -> 16 composants. Restent le S3, le nRF24, leurs découplages, le
  connecteur de prog et les 100 ohms. Partis : la matrice 26 switchs / 24
  diodes, les 11 TVS, le TRRS, l'écran, le trackpad.
- usbc : 6 -> 4 composants. Le hub CH334R (U53) est parti, il venait du coffre
  P4 et n'avait rien à faire dans une souris. Restent J48, U54 (USBLC6) et les
  deux 5k1 de CC.

Tables de bibliothèques réparées : elles pointaient vers des fichiers absents ou
renommés (optical mouse.lib -> optical_mouse.lib, nice_nano, RP2040, SSD1306).
Mouse.pretty rapatrié du fork : les 6 empreintes de la coque en dépendent.

ERC : 96 -> 24 violations.

Co-Authored-By: Claude Opus 5 <noreply@anthropic.com>
Claude-Session: https://claude.ai/code/session_01GfX5RmekmQi78Dm37qsT4Z
Parts:
- removed C53: 10uF, Capacitor_SMD:C_1206_3216Metric_Pad1.33x1.80mm_HandSolder, symbol Device:C
- removed U53: CH334R, Package_SO:QSOP-16_3.9x4.9mm_P0.635mm, symbol Interface_USB:CH334R
Connections:
- net DPU+ is gone; now on net D+_s3: U54.4 (I/O2)
- net DPU- is gone; now on net D-_s3: U54.6 (I/O1)
- no-connect marks 6 -> 2
