File: hardware/pcb/power.kicad_sch (KiCad schematic)
At the start: 22 parts, among them J10 Battery, Q2 AO3407, Q4 FS8205, SW54 SW_SPDT, U18 TP4056-42-ESOP8, U20 HT7833, U23 DW01A

Commit message: logos Niphargus importés dans la bibliothèque
Les 5 empreintes de logo vivaient seulement dans le MaeLid du clavier — le
MaeLid de Conchodytes venait du fork Mouse, qui ne contient que D_SOD-123 et
LOGO. Même cause que le nRF24 manquant au premier F8.

Copiées : Niphargus_10mm_Cu et _silk (8,8 x 9,0 mm — la crevette),
niphargus_19mm_silk (17,7 x 18,1), Niphargus_text_3mm_Cu et _silk
(15,6 x 3,9 — le mot). Sur le clavier, HS1/HS2 utilisent la version cuivre au
dos et HS3 le texte en sérigraphie à l'avant.

Rien n'est posé sur la carte : Mae les placera elle-même. fp-lib-table
inchangée, MaeLid y était déjà déclarée et reste résolue.

Co-Authored-By: Claude Opus 5 <noreply@anthropic.com>
Claude-Session: https://claude.ai/code/session_01GfX5RmekmQi78Dm37qsT4Z
Connections:
- net at Q2.2 (S): now also SW54.3 (C); no longer SW54.2 (B)
- net at C24.2, D52.1 (K), U20.2 (VI): now also SW54.2 (B); no longer SW54.3 (C)
Other:
- moved on the sheet: SW54
Changed lines of the file:
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@@
 	)
 	(no_connect
-		(at 68.58 165.1)
+		(at 55.88 170.18)
 	)
 	(wire
@@
 	(wire
 		(pts
+			(xy 66.04 167.64) (xy 66.04 170.18)
+		)
+		(stroke
+			(width 0)
+			(type default)
+		)
+	)
+	(wire
+		(pts
 			(xy 34.29 69.85) (xy 34.29 87.63)
 		)
@@
 	(wire
 		(pts
+			(xy 55.88 165.1) (xy 55.88 167.64)
+		)
+		(stroke
+			(width 0)
+			(type default)
+		)
+	)
+	(wire
+		(pts
 			(xy 29.21 104.14) (xy 29.21 107.95)
 		)
@@
 		(pts
 			(xy 30.48 184.15) (xy 30.48 167.64)
-		)
-		(stroke
-			(width 0)
-			(type default)
-		)
-	)
-	(wire
-		(pts
-			(xy 68.58 165.1) (xy 66.04 165.1)
 		)
 		(stroke
@@
 	(symbol
 		(lib_id "Switch:SW_SPDT")
-		(at 60.96 167.64 0)
+		(at 60.96 167.64 180)
 		(unit 1)
 		(body_style 1)
@@
 		)
 		(property "Datasheet" ""
-			(at 60.96 175.26 0)
-			(hide yes)
-			(show_name no)
+			(at 60.96 160.02 0)
+			(hide yes)
+			(show_name no)
